File: copam.kicad_pcb (KiCad board)
At the start: 2 copper layers, 428.6 x 142.9 mm, 193 parts, among them K0:0 KEYSW, K0:1 KEYSW, K0:2 KEYSW, K0:3 KEYSW, K0:4 KEYSW, K10:0 KEYSW, K10:1 KEYSW, K10:2 KEYSW, K10:3 KEYSW, K11:0 KEYSW, K11:1 KEYSW, K11:2 KEYSW, K11:3 KEYSW, K12:0 KEYSW, K12:1 KEYSW, K12:2 KEYSW, K12:3 KEYSW, K13:0 KEYSW, K13:1 KEYSW, K13:2 KEYSW, K13:4 KEYSW, K14:0 KEYSW, K14:1 KEYSW, K14:4 KEYSW, K15:0 KEYSW, K15:0_1 KEYSW, K15:4 KEYSW, K16:0 KEYSW, K16:1 KEYSW, K16:2 KEYSW, K16:3 KEYSW, K16:4 KEYSW, K16:4_1 KEYSW, K17:0 KEYSW, K17:1 KEYSW, K17:2 KEYSW, K17:3 KEYSW, K17:4 KEYSW, K18:0 KEYSW, K18:1 KEYSW, K18:2 KEYSW, K18:3 KEYSW, K19:0 KEYSW, K19:1 KEYSW, K19:2 KEYSW, K19:3 KEYSW, K19:4 KEYSW, K1:0 KEYSW, K1:1 KEYSW, K1:2 KEYSW, K1:3 KEYSW, K1:4 KEYSW, K20:0 KEYSW, K20:1 KEYSW, K20:2 KEYSW, K20:4 KEYSW, K2:0 KEYSW, K2:1 KEYSW, K2:2 KEYSW, K2:2_1 KEYSW, K2:3 KEYSW, K2:4 KEYSW, K3:0 KEYSW, K3:1 KEYSW, K3:2 KEYSW, K3:3 KEYSW, K3:4 KEYSW, K47 KEYSW, K4:0 KEYSW, K4:1 KEYSW, K4:2 KEYSW, K4:3 KEYSW, K5:0 KEYSW, K5:1 KEYSW, K5:2 KEYSW, K5:3 KEYSW, K6:0 KEYSW, K6:1 KEYSW, K6:2 KEYSW, K6:3 KEYSW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

Commit message: Migration to Kicad 6
Parts:
- removed ?: , Keyboard_Footprints:USB_Mini-B_SMD
- removed D10:0, D10:1, D10:2, D10:3, D11:0, D11:1, D11:2, D11:3, D12:0, D12:1, D12:2, D12:3, D13:0, D13:1, D13:2, D13:4, D14:0, D14:1, D14:4, D15:0, D15:4, D16:0, D16:1, D16:2, D16:3, D16:4, D17:0, D17:1, D17:2, D17:3, D17:4, D18:0, D18:1, D18:2, D18:3, D19:0, D19:1, D19:2, D19:3, D19:4, D20:0, D20:1, D20:2, D20:4, D5:0, D5:1, D5:2, D5:3, D6:0, D6:1, D6:2, D6:3, D7:0, D7:1, D7:2, D7:3, D7:4, D8:0, D8:1, D8:2, D8:3, D9:0, D9:1, D9:2, D9:3: D, Keyboard_Footprints:Diode_123
- removed K10:0, K10:1, K10:2, K10:3, K11:0, K11:1, K11:2, K11:3, K12:0, K12:1, K12:2, K12:3, K13:0, K13:1, K13:2, K13:4, K14:0, K14:1, K14:4, K15:0, K15:0_1, K15:4, K16:0, K16:1, K16:2, K16:3, K16:4, K16:4_1, K17:0, K17:1, K17:2, K17:3, K17:4, K18:0, K18:1, K18:2, K18:3, K19:0, K19:1, K19:2, K19:3, K19:4, K20:0, K20:1, K20:2, K20:4, K5:0, K5:1, K5:2, K5:3, K6:0, K6:1, K6:2, K6:3, K7:0, K7:1, K7:2, K7:3, K7:4, K8:0, K8:1, K8:2, K8:3, K9:0, K9:1, K9:2, K9:3: KEYSW, Keyboard_Footprints:Alps_Hotswap
- removed K47: KEYSW, Keyboard_Footprints:Alps_Hotswap_Hasu
- removed LEDA1, LEDB1, LEDC1: LED, Keyboard_Footprints:LED_Rectangular_W3.9mm_H1.8mm_FlatTop
- removed RA1, RB1, RC1: R, Resistors_SMD:R_0805_HandSoldering
- removed USB: , Pin_Headers:Pin_Header_Straight_1x05_Pitch2.00mm
- added D0:10: D, Diode_SMD:D_SOD-123, B.Cu at (242.9, 78.6)
- added D0:11: D, Diode_SMD:D_SOD-123, B.Cu at (261.9, 78.6)
- added D0:12: D, Diode_SMD:D_SOD-123, B.Cu at (281.0, 78.6)
- added D0:13: D, Diode_SMD:D_SOD-123, B.Cu at (300.0, 78.6)
- added D0:14: D, Diode_SMD:D_SOD-123, B.Cu at (319.1, 78.6)
- added D0:15: D, Diode_SMD:D_SOD-123, B.Cu at (338.1, 78.6)
- added D0:16: D, Diode_SMD:D_SOD-123, B.Cu at (357.2, 78.6)
- added D0:17: D, Diode_SMD:D_SOD-123, B.Cu at (385.8, 78.6)
- added D0:18: D, Diode_SMD:D_SOD-123, B.Cu at (404.8, 78.6)
- added D0:19: D, Diode_SMD:D_SOD-123, B.Cu at (423.9, 78.6)
- added D0:20: D, Diode_SMD:D_SOD-123, B.Cu at (442.9, 78.6)
- added D0:5: D, Diode_SMD:D_SOD-123, B.Cu at (147.6, 78.6)
- added D0:6: D, Diode_SMD:D_SOD-123, B.Cu at (166.7, 78.6)
- added D0:7: D, Diode_SMD:D_SOD-123, B.Cu at (185.7, 78.6)
- added D0:8: D, Diode_SMD:D_SOD-123, B.Cu at (204.8, 78.6)
- added D0:9: D, Diode_SMD:D_SOD-123, B.Cu at (223.8, 78.6)
- added D1:10: D, Diode_SMD:D_SOD-123, B.Cu at (252.4, 97.6)
- added D1:11: D, Diode_SMD:D_SOD-123, B.Cu at (271.5, 97.6)
- added D1:12: D, Diode_SMD:D_SOD-123, B.Cu at (290.5, 97.6)
- added D1:13: D, Diode_SMD:D_SOD-123, B.Cu at (309.6, 97.6)
- added D1:14: D, Diode_SMD:D_SOD-123, B.Cu at (328.6, 97.6)
- added D1:16: D, Diode_SMD:D_SOD-123, B.Cu at (352.4, 97.6)
- added D1:17: D, Diode_SMD:D_SOD-123, B.Cu at (385.7, 97.6)
- added D1:18: D, Diode_SMD:D_SOD-123, B.Cu at (404.8, 97.6)
- added D1:19: D, Diode_SMD:D_SOD-123, B.Cu at (423.8, 97.6)
- added D1:20: D, Diode_SMD:D_SOD-123, B.Cu at (442.9, 97.6)
- added D1:5: D, Diode_SMD:D_SOD-123, B.Cu at (157.2, 97.6)
- added D1:6: D, Diode_SMD:D_SOD-123, B.Cu at (176.2, 97.6)
- added D1:7: D, Diode_SMD:D_SOD-123, B.Cu at (195.3, 97.6)
- added D1:8: D, Diode_SMD:D_SOD-123, B.Cu at (214.3, 97.6)
- added D1:9: D, Diode_SMD:D_SOD-123, B.Cu at (233.4, 97.6)
- added D2:10: D, Diode_SMD:D_SOD-123, B.Cu at (257.1, 116.7)
- added D2:11: D, Diode_SMD:D_SOD-123, B.Cu at (276.2, 116.7)
- added D2:12: D, Diode_SMD:D_SOD-123, B.Cu at (295.2, 116.7)
- added D2:13: D, Diode_SMD:D_SOD-123, B.Cu at (314.3, 116.7)
- added D2:16: D, Diode_SMD:D_SOD-123, B.Cu at (345.3, 116.7)
- added D2:17: D, Diode_SMD:D_SOD-123, B.Cu at (385.7, 116.7)
- added D2:18: D, Diode_SMD:D_SOD-123, B.Cu at (404.8, 116.7)
- added D2:19: D, Diode_SMD:D_SOD-123, B.Cu at (423.8, 116.7)
- added D2:20: D, Diode_SMD:D_SOD-123, B.Cu at (442.9, 116.7)
- added D2:5: D, Diode_SMD:D_SOD-123, B.Cu at (161.9, 116.7)
- added D2:6: D, Diode_SMD:D_SOD-123, B.Cu at (181.0, 116.7)
- added D2:7: D, Diode_SMD:D_SOD-123, B.Cu at (200.0, 116.7)
- added D2:8: D, Diode_SMD:D_SOD-123, B.Cu at (219.1, 116.7)
- added D2:9: D, Diode_SMD:D_SOD-123, B.Cu at (238.1, 116.7)
- added D3:10: D, Diode_SMD:D_SOD-123, B.Cu at (266.7, 135.7)
- added D3:11: D, Diode_SMD:D_SOD-123, B.Cu at (285.7, 135.7)
- added D3:12: D, Diode_SMD:D_SOD-123, B.Cu at (304.8, 135.7)
- added D3:16: D, Diode_SMD:D_SOD-123, B.Cu at (340.5, 135.7)
- added D3:17: D, Diode_SMD:D_SOD-123, B.Cu at (385.8, 135.7)
- added D3:18: D, Diode_SMD:D_SOD-123, B.Cu at (404.8, 135.7)
- added D3:19: D, Diode_SMD:D_SOD-123, B.Cu at (423.9, 135.7)
- added D3:5: D, Diode_SMD:D_SOD-123, B.Cu at (171.4, 135.7)
- added D3:6: D, Diode_SMD:D_SOD-123, B.Cu at (190.5, 135.7)
- added D3:7: D, Diode_SMD:D_SOD-123, B.Cu at (209.6, 135.7)
- added D3:8: D, Diode_SMD:D_SOD-123, B.Cu at (228.6, 135.7)
- added D3:9: D, Diode_SMD:D_SOD-123, B.Cu at (247.6, 135.7)
- added D4:13: D, Diode_SMD:D_SOD-123, B.Cu at (300.0, 154.8)
- added D4:14: D, Diode_SMD:D_SOD-123, B.Cu at (319.1, 154.8)
- added D4:15: D, Diode_SMD:D_SOD-123, B.Cu at (338.1, 154.8)
- added D4:16: D, Diode_SMD:D_SOD-123, B.Cu at (357.2, 154.8)
- added D4:17: D, Diode_SMD:D_SOD-123, B.Cu at (395.3, 154.8)
- added D4:19: D, Diode_SMD:D_SOD-123, B.Cu at (423.9, 154.8)
- added D4:20: D, Diode_SMD:D_SOD-123, B.Cu at (438.1, 154.8)
- added D4:7: D, Diode_SMD:D_SOD-123, B.Cu at (214.3, 154.8)
- added K0:10: KEYSW, Keyboard_Footprints:Alps_Hotswap, F.Cu at (238.1, 76.2)
- added K0:11: KEYSW, Keyboard_Footprints:Alps_Hotswap, F.Cu at (257.1, 76.2)
- added K0:12: KEYSW, Keyboard_Footprints:Alps_Hotswap, F.Cu at (276.2, 76.2)
- added K0:13: KEYSW, Keyboard_Footprints:Alps_Hotswap, F.Cu at (295.2, 76.2)
- added K0:14: KEYSW, Keyboard_Footprints:Alps_Hotswap, F.Cu at (314.3, 76.2)
- added K0:15: KEYSW, Keyboard_Footprints:Alps_Hotswap, F.Cu at (333.4, 76.2)
- added K0:15_1: KEYSW, Keyboard_Footprints:Alps_Hotswap_Secondary, F.Cu at (342.9, 76.2)
- added K0:16: KEYSW, Keyboard_Footprints:Alps_Hotswap, F.Cu at (352.4, 76.2)
- added K0:17: KEYSW, Keyboard_Footprints:Alps_Hotswap, F.Cu at (380.9, 76.2)
- added K0:18: KEYSW, Keyboard_Footprints:Alps_Hotswap, F.Cu at (400.0, 76.2)
- added K0:19: KEYSW, Keyboard_Footprints:Alps_Hotswap, F.Cu at (419.1, 76.2)
- added K0:20: KEYSW, Keyboard_Footprints:Alps_Hotswap, F.Cu at (438.1, 76.2)
- added K0:5: KEYSW, Keyboard_Footprints:Alps_Hotswap, F.Cu at (142.8, 76.2)
- added K0:6: KEYSW, Keyboard_Footprints:Alps_Hotswap, F.Cu at (161.9, 76.2)
- added K0:7: KEYSW, Keyboard_Footprints:Alps_Hotswap, F.Cu at (180.9, 76.2)
- added K0:8: KEYSW, Keyboard_Footprints:Alps_Hotswap, F.Cu at (200.0, 76.2)
- added K0:9: KEYSW, Keyboard_Footprints:Alps_Hotswap, F.Cu at (219.1, 76.2)
- added K1:10: KEYSW, Keyboard_Footprints:Alps_Hotswap, F.Cu at (247.6, 95.2)
- added K1:11: KEYSW, Keyboard_Footprints:Alps_Hotswap, F.Cu at (266.7, 95.2)
- added K1:12: KEYSW, Keyboard_Footprints:Alps_Hotswap, F.Cu at (285.7, 95.2)
- added K1:13: KEYSW, Keyboard_Footprints:Alps_Hotswap, F.Cu at (304.8, 95.2)
- added K1:14: KEYSW, Keyboard_Footprints:Alps_Hotswap, F.Cu at (323.8, 95.2)
- added K1:16: KEYSW, Keyboard_Footprints:Alps_Hotswap, F.Cu at (347.7, 95.2)
- added K1:17: KEYSW, Keyboard_Footprints:Alps_Hotswap, F.Cu at (380.9, 95.2)
- added K1:18: KEYSW, Keyboard_Footprints:Alps_Hotswap, F.Cu at (400.0, 95.2)
- added K1:19: KEYSW, Keyboard_Footprints:Alps_Hotswap, F.Cu at (419.1, 95.2)
- added K1:20: KEYSW, Keyboard_Footprints:Alps_Hotswap, F.Cu at (438.1, 95.2)
- added K1:5: KEYSW, Keyboard_Footprints:Alps_Hotswap, F.Cu at (152.4, 95.2)
- added K1:6: KEYSW, Keyboard_Footprints:Alps_Hotswap, F.Cu at (171.4, 95.2)
- added K1:7: KEYSW, Keyboard_Footprints:Alps_Hotswap, F.Cu at (190.5, 95.2)
- added K1:8: KEYSW, Keyboard_Footprints:Alps_Hotswap, F.Cu at (209.5, 95.2)
- added K1:9: KEYSW, Keyboard_Footprints:Alps_Hotswap, F.Cu at (228.6, 95.2)
- added K2:10: KEYSW, Keyboard_Footprints:Alps_Hotswap, F.Cu at (252.4, 114.3)
- added K2:11: KEYSW, Keyboard_Footprints:Alps_Hotswap, F.Cu at (271.4, 114.3)
- added K2:12: KEYSW, Keyboard_Footprints:Alps_Hotswap, F.Cu at (290.5, 114.3)
- added K2:13: KEYSW, Keyboard_Footprints:Alps_Hotswap, F.Cu at (309.5, 114.3)
- added K2:16: KEYSW, Keyboard_Footprints:Alps_Hotswap, F.Cu at (340.5, 114.3)
- added K2:17: KEYSW, Keyboard_Footprints:Alps_Hotswap, F.Cu at (380.9, 114.3)
- added K2:18: KEYSW, Keyboard_Footprints:Alps_Hotswap, F.Cu at (400.0, 114.3)
- added K2:19: KEYSW, Keyboard_Footprints:Alps_Hotswap, F.Cu at (419.1, 114.3)
- added K2:20: KEYSW, Keyboard_Footprints:Alps_Hotswap, F.Cu at (438.1, 114.3)
- added K2:5: KEYSW, Keyboard_Footprints:Alps_Hotswap, F.Cu at (157.1, 114.3)
- added K2:6: KEYSW, Keyboard_Footprints:Alps_Hotswap, F.Cu at (176.2, 114.3)
- added K2:7: KEYSW, Keyboard_Footprints:Alps_Hotswap, F.Cu at (195.2, 114.3)
- added K2:8: KEYSW, Keyboard_Footprints:Alps_Hotswap, F.Cu at (214.3, 114.3)
- added K2:9: KEYSW, Keyboard_Footprints:Alps_Hotswap, F.Cu at (233.3, 114.3)
- added K3:10: KEYSW, Keyboard_Footprints:Alps_Hotswap, F.Cu at (261.9, 133.3)
- added K3:11: KEYSW, Keyboard_Footprints:Alps_Hotswap, F.Cu at (281.0, 133.3)
- added K3:12: KEYSW, Keyboard_Footprints:Alps_Hotswap, F.Cu at (300.0, 133.3)
- added K3:16: KEYSW, Keyboard_Footprints:Alps_Hotswap, F.Cu at (335.7, 133.3)
- added K3:17: KEYSW, Keyboard_Footprints:Alps_Hotswap, F.Cu at (380.9, 133.3)
- added K3:18: KEYSW, Keyboard_Footprints:Alps_Hotswap, F.Cu at (400.0, 133.3)
- added K3:19: KEYSW, Keyboard_Footprints:Alps_Hotswap, F.Cu at (419.1, 133.3)
- added K3:5: KEYSW, Keyboard_Footprints:Alps_Hotswap, F.Cu at (166.7, 133.3)
- added K3:6: KEYSW, Keyboard_Footprints:Alps_Hotswap, F.Cu at (185.7, 133.3)
- added K3:7: KEYSW, Keyboard_Footprints:Alps_Hotswap, F.Cu at (204.8, 133.3)
- added K3:8: KEYSW, Keyboard_Footprints:Alps_Hotswap, F.Cu at (223.8, 133.3)
- added K3:9: KEYSW, Keyboard_Footprints:Alps_Hotswap, F.Cu at (242.9, 133.3)
- added K4:13: KEYSW, Keyboard_Footprints:Alps_Hotswap, F.Cu at (295.2, 152.4)
- added K4:14: KEYSW, Keyboard_Footprints:Alps_Hotswap, F.Cu at (314.3, 152.4)
- added K4:15: KEYSW, Keyboard_Footprints:Alps_Hotswap, F.Cu at (333.4, 152.4)
- added K4:16: KEYSW, Keyboard_Footprints:Alps_Hotswap, F.Cu at (352.4, 152.4)
- added K4:16_1: KEYSW, Keyboard_Footprints:Alps_Hotswap_Secondary, F.Cu at (347.7, 152.4)
- added K4:17: KEYSW, Keyboard_Footprints:Alps_Hotswap, F.Cu at (390.5, 152.4)
- added K4:19: KEYSW, Keyboard_Footprints:Alps_Hotswap, F.Cu at (419.1, 152.4)
- added K4:20: KEYSW, Keyboard_Footprints:Alps_Hotswap, F.Cu at (438.1, 142.9)
- added K4:7: KEYSW, Keyboard_Footprints:Alps_Hotswap, F.Cu at (209.5, 152.4)
- added LED1: 5mm_Rectangular, LED_THT:LED_Rectangular_W5.0mm_H2.0mm, F.Cu at (349.5, 45.5)
- added LED2: 5mm_Rectangular, LED_THT:LED_Rectangular_W5.0mm_H2.0mm, F.Cu at (386.2, 45.5)
- added LED3: 5mm_Rectangular, LED_THT:LED_Rectangular_W5.0mm_H2.0mm, F.Cu at (423.0, 45.5)
- added R1: R, Resistor_SMD:R_0805_2012Metric, B.Cu at (358.2, 45.5)
- added R2: R, Resistor_SMD:R_0805_2012Metric, B.Cu at (395.0, 45.5)
- added R3: R, Resistor_SMD:R_0805_2012Metric, B.Cu at (431.8, 45.5)
- D0:0, D0:1, D0:2, D0:3, D0:4, D1:0, D1:1, D1:2, D1:3, D1:4, D2:0, D2:1, D2:2, D2:3, D2:4, D3:0, D3:1, D3:2, D3:3, D3:4, D4:0, D4:1, D4:2, D4:3: footprint Keyboard_Footprints:Diode_123 -> Diode_SMD:D_SOD-123; moved to B.Cu
- J1: value (none) -> CONN_01X02; footprint Pin_Headers:Pin_Header_Straight_1x02_Pitch2.00mm -> Connector_PinHeader_2.00mm:PinHeader_1x02_P2.00mm_Vertical
- K2:2_1: footprint Keyboard_Footprints:Alps_Hotswap -> Keyboard_Footprints:Alps_Hotswap_Secondary
- SW1: value (none) -> SW_PUSH; footprint Keyboard_Footprints:Copam_Reset -> Keyboard_Footprints:TE_1825966-1
- moved D0:4 120.5 mm to (128.6, 78.6), turned to 90 degrees
- moved K0:4 115.3 mm to (123.8, 76.2)
- moved K4:0 114.5 mm to (38.1, 152.4)
- moved D4:0 109.4 mm to (42.9, 154.8), turned to 90 degrees
- moved D1:4 101.7 mm to (138.1, 97.6), turned to 90 degrees
- moved K1:4 96.4 mm to (133.3, 95.2)
- moved K4:1 94.5 mm to (57.1, 152.4)
- moved D0:3 93.8 mm to (109.5, 78.6), turned to 90 degrees
- moved D4:1 89.4 mm to (61.9, 154.8), turned to 90 degrees
- moved K0:3 88.6 mm to (104.8, 76.2)
- moved K3:0 87.5 mm to (38.1, 133.3)
- moved D3:0 82.5 mm to (42.9, 135.7), turned to 90 degrees
- moved D1:3 75.6 mm to (119.1, 97.6), turned to 90 degrees
- moved K1:3 70.3 mm to (114.3, 95.2)
- moved K3:1 67.7 mm to (57.1, 133.3)
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Connections:
- D0:1 pad 1: Net-(D0:1-Pad1) -> Net-(D0:0-Pad1)
- D0:2 pad 1: Net-(D0:2-Pad1) -> Net-(D0:0-Pad1)
- D0:3 pad 1: Net-(D0:3-Pad1) -> Net-(D0:0-Pad1)
- D0:4 pad 1: Net-(D0:4-Pad1) -> Net-(D0:0-Pad1)
- D1:0 pad 1: Net-(D0:0-Pad1) -> Net-(D1:0-Pad1)
- D1:1 pad 1: Net-(D0:1-Pad1) -> Net-(D1:0-Pad1)
- D1:2 pad 1: Net-(D0:2-Pad1) -> Net-(D1:0-Pad1)
- D1:3 pad 1: Net-(D0:3-Pad1) -> Net-(D1:0-Pad1)
- D1:4 pad 1: Net-(D0:4-Pad1) -> Net-(D1:0-Pad1)
- D2:0 pad 1: Net-(D0:0-Pad1) -> Net-(D2:0-Pad1)
- D2:1 pad 1: Net-(D0:1-Pad1) -> Net-(D2:0-Pad1)
- D2:2 pad 1: Net-(D0:2-Pad1) -> Net-(D2:0-Pad1)
- D2:3 pad 1: Net-(D0:3-Pad1) -> Net-(D2:0-Pad1)
- D2:4 pad 1: Net-(D0:4-Pad1) -> Net-(D2:0-Pad1)
- D3:0 pad 1: Net-(D0:0-Pad1) -> Net-(D3:0-Pad1)
- D3:1 pad 1: Net-(D0:1-Pad1) -> Net-(D3:0-Pad1)
- D3:2 pad 1: Net-(D0:2-Pad1) -> Net-(D3:0-Pad1)
- D3:3 pad 1: Net-(D0:3-Pad1) -> Net-(D3:0-Pad1)
- D3:4 pad 1: Net-(D0:4-Pad1) -> Net-(D3:0-Pad1)
- D4:0 pad 1: Net-(D0:0-Pad1) -> Net-(D4:0-Pad1)
- D4:1 pad 1: Net-(D0:1-Pad1) -> Net-(D4:0-Pad1)
- D4:2 pad 1: Net-(D0:2-Pad1) -> Net-(D4:0-Pad1)
- D4:3 pad 1: Net-(D0:3-Pad1) -> Net-(D4:0-Pad1)
- K0:1 pad 1: Net-(K0:0-Pad1) -> Net-(K0:1-Pad1)
- K0:2 pad 1: Net-(K0:0-Pad1) -> Net-(K0:2-Pad1)
- K0:3 pad 1: Net-(K0:0-Pad1) -> Net-(K0:3-Pad1)
- K0:4 pad 1: Net-(K0:0-Pad1) -> Net-(K0:4-Pad1)
- K1:0 pad 1: Net-(K1:0-Pad1) -> Net-(K0:0-Pad1)
- K1:1 pad 1: Net-(K1:0-Pad1) -> Net-(K0:1-Pad1)
- K1:2 pad 1: Net-(K1:0-Pad1) -> Net-(K0:2-Pad1)
- K1:3 pad 1: Net-(K1:0-Pad1) -> Net-(K0:3-Pad1)
- K1:4 pad 1: Net-(K1:0-Pad1) -> Net-(K0:4-Pad1)
- K2:0 pad 1: Net-(K2:0-Pad1) -> Net-(K0:0-Pad1)
- K2:1 pad 1: Net-(K2:0-Pad1) -> Net-(K0:1-Pad1)
- K2:2 pad 1: Net-(K2:0-Pad1) -> Net-(K0:2-Pad1)
- K2:2_1 pad 1: Net-(K2:0-Pad1) -> Net-(K0:2-Pad1)
- K2:3 pad 1: Net-(K2:0-Pad1) -> Net-(K0:3-Pad1)
- K2:4 pad 1: Net-(K2:0-Pad1) -> Net-(K0:4-Pad1)
- K3:0 pad 1: Net-(K3:0-Pad1) -> Net-(K0:0-Pad1)
- K3:1 pad 1: Net-(K3:0-Pad1) -> Net-(K0:1-Pad1)
- K3:2 pad 1: Net-(K3:0-Pad1) -> Net-(K0:2-Pad1)
- K3:3 pad 1: Net-(K3:0-Pad1) -> Net-(K0:3-Pad1)
- K3:4 pad 1: Net-(K3:0-Pad1) -> Net-(K0:4-Pad1)
- K4:0 pad 1: Net-(K4:0-Pad1) -> Net-(K0:0-Pad1)
- K4:1 pad 1: Net-(K4:0-Pad1) -> Net-(K0:1-Pad1)
- K4:2 pad 1: Net-(K4:0-Pad1) -> Net-(K0:2-Pad1)
- K4:3 pad 1: Net-(K4:0-Pad1) -> Net-(K0:3-Pad1)
- U1 pad 12: Net-(K1:0-Pad1) -> Net-(K0:1-Pad1)
- U1 pad 13: Net-(K2:0-Pad1) -> Net-(K0:2-Pad1)
- U1 pad 14: Net-(K3:0-Pad1) -> Net-(K0:3-Pad1)
- U1 pad 15: Net-(K4:0-Pad1) -> Net-(K0:4-Pad1)
- U1 pad 19: Net-(U1-Pad19) -> unconnected-(U1-Pad19)
- U1 pad 20: Net-(U1-Pad20) -> unconnected-(U1-Pad20)
- U1 pad 29: Net-(U1-Pad29) -> unconnected-(U1-Pad29)
- U1 pad 3: Net-(D0:4-Pad1) -> Net-(D4:0-Pad1)
- U1 pad 30: Net-(U1-Pad30) -> unconnected-(U1-Pad30)
- U1 pad 31: Net-(U1-Pad31) -> unconnected-(U1-Pad31)
- U1 pad 32: Net-(U1-Pad32) -> unconnected-(U1-Pad32)
- U1 pad 4: Net-(D0:3-Pad1) -> Net-(D3:0-Pad1)
- U1 pad 40: Net-(U1-Pad40) -> unconnected-(U1-Pad40)
- U1 pad 41: Net-(U1-Pad41) -> unconnected-(U1-Pad41)
- U1 pad 42: Net-(U1-Pad42) -> unconnected-(U1-Pad42)
- U1 pad 43: Net-(U1-Pad43) -> unconnected-(U1-Pad43)
- U1 pad 44: Net-(U1-Pad44) -> unconnected-(U1-Pad44)
- U1 pad 45: Net-(U1-Pad45) -> unconnected-(U1-Pad45)
- U1 pad 46: Net-(U1-Pad46) -> unconnected-(U1-Pad46)
- U1 pad 47: Net-(U1-Pad47) -> unconnected-(U1-Pad47)
- U1 pad 48: Net-(U1-Pad48) -> unconnected-(U1-Pad48)
- U1 pad 49: Net-(U1-Pad49) -> unconnected-(U1-Pad49)
- U1 pad 5: Net-(J1-Pad1) -> Net-(J1-Pad2)
- U1 pad 51: Net-(U1-Pad51) -> unconnected-(U1-Pad51)
- U1 pad 6: Net-(J1-Pad2) -> Net-(J1-Pad1)
- U1 pad 7: Net-(U1-Pad7) -> unconnected-(U1-Pad7)
- U1 pad 8: Net-(D0:2-Pad1) -> Net-(D2:0-Pad1)
- U1 pad 9: Net-(D0:1-Pad1) -> Net-(D1:0-Pad1)
Routing:
- net Net-(D0:4-Pad1): track 808.4 -> 0.00 mm, vias 1 -> 0
- net Net-(D0:2-Pad1): track 784.3 -> 0.00 mm
- net Net-(D0:3-Pad1): track 784.0 -> 0.00 mm, vias 1 -> 0
- net Net-(D4:0-Pad1): track 0.00 -> 777.9 mm
- net Net-(D2:0-Pad1): track 0.00 -> 751.1 mm
- net Net-(D3:0-Pad1): track 0.00 -> 748.6 mm
- net Net-(D1:0-Pad1): track 0.00 -> 579.6 mm
- net Net-(D0:1-Pad1): track 575.6 -> 0.00 mm, vias 1 -> 0
- net Net-(K0:1-Pad1): track 0.00 -> 187.6 mm
- net Net-(K0:2-Pad1): track 0.00 -> 176.8 mm
- net Net-(K1:0-Pad1): track 176.8 -> 0.00 mm, vias 1 -> 0
- net Net-(K2:0-Pad1): track 172.8 -> 0.00 mm, vias 1 -> 0
- net Net-(K0:3-Pad1): track 0.00 -> 155.2 mm
- net Net-(K3:0-Pad1): track 148.6 -> 0.00 mm, vias 1 -> 0
- net (no net): track 130.2 -> 0.00 mm, vias 5 -> 0
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Other:
- board size 428.6 x 142.9 mm -> 428 x 147 mm
- net class D2 removed
- net class D3 removed
- net class Default removed
